Commit message: Increase BRUCE URDF joint effort and velocity limits

File: resources/robots/bruce/bruce.urdf (robot description, URDF)
Before this commit: robot bruce, 17 links, 16 joints
Joints:
- joint ankle_pitch_l: limit lower=-1.50 upper=1.50 effort=10.5 velocity=20.0 -> lower=-1.50 upper=1.50 effort=31.5 velocity=60.0
- joint ankle_pitch_r: limit lower=-1.50 upper=1.50 effort=10.5 velocity=20.0 -> lower=-1.50 upper=1.50 effort=31.5 velocity=60.0
- joint elbow_pitch_l: limit lower=-2.30 upper=2.30 effort=10.5 velocity=20.0 -> lower=-2.30 upper=2.30 effort=31.5 velocity=60.0
- joint elbow_pitch_r: limit lower=-2.30 upper=2.30 effort=10.5 velocity=20.0 -> lower=-2.30 upper=2.30 effort=31.5 velocity=60.0
- joint hip_pitch_l: limit lower=-0.40 upper=2.50 effort=10.5 velocity=20.0 -> lower=-0.40 upper=2.50 effort=31.5 velocity=60.0
- joint hip_pitch_r: limit lower=-0.40 upper=2.50 effort=10.5 velocity=20.0 -> lower=-0.40 upper=2.50 effort=31.5 velocity=60.0
- joint hip_roll_l: limit lower=-0.78539816339 upper=0.78539816339 effort=10.5 velocity=20.0 -> lower=-0.78539816339 upper=0.78539816339 effort=31.5 velocity=60.0
- joint hip_roll_r: limit lower=-0.78539816339 upper=0.78539816339 effort=10.5 velocity=20.0 -> lower=-0.78539816339 upper=0.78539816339 effort=31.5 velocity=60.0
- joint hip_yaw_l: limit lower=-1.57079632679 upper=1.57079632679 effort=10.5 velocity=20.0 -> lower=-1.57079632679 upper=1.57079632679 effort=31.5 velocity=60.0
- joint hip_yaw_r: limit lower=-1.57079632679 upper=1.57079632679 effort=10.5 velocity=20.0 -> lower=-1.57079632679 upper=1.57079632679 effort=31.5 velocity=60.0
- joint knee_pitch_l: limit lower=-2.50 upper=-0.01 effort=10.5 velocity=20.0 -> lower=-2.50 upper=-0.01 effort=31.5 velocity=60.0
- joint knee_pitch_r: limit lower=-2.50 upper=-0.01 effort=10.5 velocity=20.0 -> lower=-2.50 upper=-0.01 effort=31.5 velocity=60.0
- joint shoulder_pitch_l: limit lower=-3.14159265359 upper=3.14159265359 effort=10.5 velocity=20.0 -> lower=-3.14159265359 upper=3.14159265359 effort=31.5 velocity=60.0
- joint shoulder_pitch_r: limit lower=-3.14159265359 upper=3.14159265359 effort=10.5 velocity=20.0 -> lower=-3.14159265359 upper=3.14159265359 effort=31.5 velocity=60.0
- joint shoulder_roll_l: limit lower=-1.90 upper=1.57079632679 effort=10.5 velocity=20.0 -> lower=-1.90 upper=1.57079632679 effort=31.5 velocity=60.0
- joint shoulder_roll_r: limit lower=-1.57079632679 upper=1.90 effort=10.5 velocity=20.0 -> lower=-1.57079632679 upper=1.90 effort=31.5 velocity=60.0

Commit message: Flip BRUCE knee joint axis and default pose sign

File: resources/robots/bruce/bruce.urdf (robot description, URDF)
Before this commit: robot bruce, 17 links, 16 joints
Joints:
- joint knee_pitch_l: axis 0 0 1 -> 0 0 -1; limit lower=-2.50 upper=-0.01 effort=31.5 velocity=60.0 -> lower=0.01 upper=2.50 effort=31.5 velocity=60.0
- joint knee_pitch_r: axis 0 0 1 -> 0 0 -1; limit lower=-2.50 upper=-0.01 effort=31.5 velocity=60.0 -> lower=0.01 upper=2.50 effort=31.5 velocity=60.0
